File: Electrical.sch (EAGLE design)
At the start: 70 parts

Commit message: test changes for tutorial
Connections:
- new net VT10: U$38.10
- new net VT11: U$38.11
- new net VT13: U$38.13
- new net VT14: U$38.14
- new net VT15: U$38.15
- new net VT16: U$38.16
- new net VT17: U$38.17
- new net VT18: U$38.18
- new net VT19: U$38.19
- new net VT2: U$38.2
- new net VT20: U$38.20
- new net VT21: U$38.21
- new net VT22: U$38.22
- new net VT23: U$38.23
- new net VT25: U$38.25
- new net VT26: U$38.26
- new net VT27: U$38.27
- new net VT28: U$38.28
- new net VT29: U$38.29
- new net VT3: U$38.3
- new net VT30: U$38.30
- new net VT31: U$38.31
- new net VT4: U$38.4
- new net VT5: U$38.5
- new net VT6: U$38.6
- new net VT7: U$38.7
- new net VT8: U$38.8
- new net VT9: U$38.9
- net BATTERY_P: now also U$38.32
- net VT1: now also U$38.1
- net VT12: now also U$38.12
- net VT24: now also U$38.24
Other:
- moved on the sheet: U$36, U$37
