File: Aux_System.sch (EAGLE design)
At the start: 26 parts

Commit message: Auxiliary low-voltage system schematic
Parts:
- added U$17, U$18, U$19: FUSE, Solar array design :FUSE
- U$1: value DC_DC_CONVERTER -> FUSE; device Small_Scale_System - Copy:DC_DC_CONVERTER -> Solar array design :FUSE
- U$15: value USB -> FUSE; device Small_Scale_System - Copy:USB -> Solar array design :FUSE
- U$16: value CHASSIS_GND -> FUSE; device Small_Scale_System - Copy:CHASSIS_GND -> Solar array design :FUSE
Connections:
- removed net BMS_POWER: U$2.P$3, U$4.AM_PWR
- new net AUX_FUSE: U$2.P$3
- new net N$22: U$17.P$1, U$5.P$3
- new net N$26: U$18.P$1, U$5.P$6
- new net N$27: U$19.P$1, U$2.P$6
- net N$15: now also U$1.P$2, U$15.P$2, U$16.P$2, U$17.P$2, U$18.P$2, U$19.P$2; no longer HORN_RELAY.P$2, U$1.+VIN, U$11.P$1, U$2.P$1, U$2.P$6
- net N$16: now also U$8.P$5; no longer U$8.P$4
- net N$17: now also U$8.P$2; no longer U$8.P$1
- net N$18: now also U$10.P$5; no longer U$10.P$4
- net N$19: now also HORN_RELAY.P$2, U$1.P$1; no longer U$10.P$1, U$5.P$8
- net N$23: now also U$16.P$1, U$2.P$1; no longer U$1.-VOUT, U$15.V+
- net N$24: now also U$11.P$1, U$15.P$1; no longer U$15.OUT, U$16.P$1
- net N$5: now also U$10.P$2, U$5.P$8; no longer U$1.+VOUT, U$15.V-
Other:
- moved on the sheet: AUX_PWR, PRIMARY_PWR
